File: 2G4Radio.sch (KiCad schematic (older format))
At the start: 38 parts, among them P1 BNC, P2 BNC, U1 CC2520, U2 CC2592, U5 LDB182G4520C-110, X1 FA-20H32.0000MF20X-K3

Commit message: Fixed broken AVDD reference.
Routed 2.4GHz radio.
Connections:
- net VDD_CC2520_ISO: now reaches C1.1, C2.1, C4.1, C5.1, L1.1, U1.11 (AVDD1), U1.14 (AVDD2), U1.8 (DVDD)
- net VDD_CC2520_ISO: now also U1.16 (AVDD3), U1.20 (AVDD4), U1.22 (AVDD5), U1.24 (AVDD_GUARD)
- net VDD_CC2592_ISO: now reaches C10.1, C11.1, C12.1, C8.1, L2.2, L3.2, U2.13 (VDD_LNA), U2.14 (VDD_BIAS), U2.15 (VDD_PA)
- net at U1.17 (RF_P): now also R7.2; no longer R6.1
- net at U1.19 (RF_N): now also R6.2; no longer R7.1
- net at U2.2 (RF_N): now also R6.1; no longer R7.2
- net at U2.3 (RF_P): now also R7.1; no longer R6.2
- net at R7.3: now also U5.4 (BALP); no longer U5.6 (BALN)
- net at R6.3: now also U5.6 (BALN); no longer U5.4 (BALP)
Other:
- moved on the sheet: R6, R7
Changed lines of the file:
@@
 P 2650 3100
 F 0 "U1" H 2200 3750 60  0000 C CNN
-F 1 "CC2520" H 3000 3750 60  0000 C CNN
+F 1 "CC2520" H 2300 2400 60  0000 C CNN
 F 2 "SMD_Packages:RHD_S-PVQFN-N28" H 2650 3100 60  0001 C CNN
 F 3 "" H 2650 3100 60  0000 C CNN
@@
 L R3-LH R7
 U 1 1 559B6ED9
-P 5200 3350
-F 0 "R7" H 5150 3450 50  0000 C CNN
-F 1 "0" V 5450 3500 50  0000 C CNN
-F 2 "Resistors_SMD:R3_LH_0402" H 5200 3280 30  0001 C CNN
-F 3 "" V 5200 3350 30  0000 C CNN
-	1    5200 3350
-	1    0    0    -1
+P 5250 3450
+F 0 "R7" H 5200 3550 50  0000 C CNN
+F 1 "0" V 5500 3600 50  0000 C CNN
+F 2 "Resistors_SMD:R3_LH_0402" H 5250 3380 30  0001 C CNN
+F 3 "" V 5250 3450 30  0000 C CNN
+	1    5250 3450
+	-1   0    0    1
 $EndComp
 $Comp
 L R3-RH R6
 U 1 1 559B7240
-P 5200 3450
-F 0 "R6" H 5100 3350 50  0000 C CNN
-F 1 "0" V 5450 3300 50  0000 C CNN
-F 2 "Resistors_SMD:R3_RH_0402" H 5200 3380 30  0001 C CNN
-F 3 "" V 5200 3450 30  0000 C CNN
-	1    5200 3450
-	1    0    0    -1
+P 5250 3350
+F 0 "R6" H 5150 3250 50  0000 C CNN
+F 1 "0" V 5500 3200 50  0000 C CNN
+F 2 "Resistors_SMD:R3_RH_0402" H 5250 3280 30  0001 C CNN
+F 3 "" V 5250 3350 30  0000 C CNN
+	1    5250 3350
+	-1   0    0    1
 $EndComp
 $Comp
@@
 PA_EN
 NoConn ~ 2000 2550
-Wire Wire Line
-	5750 2100 8100 2100
-Wire Wire Line
-	6000 2100 6000 2150
-Wire Wire Line
-	7650 2100 7650 2150
-Connection ~ 6000 2100
-Wire Wire Line
-	7050 2150 7050 2100
-Connection ~ 7050 2100
-Wire Wire Line
-	7350 2150 7350 2100
-Connection ~ 7350 2100
-Wire Wire Line
-	8100 2100 8100 2700
-Connection ~ 7650 2100
-Wire Wire Line
-	8100 3300 8100 3600
-Wire Wire Line
-	7450 3450 8300 3450
-Connection ~ 8100 3450
-Wire Wire Line
-	8900 3450 9050 3450
-Wire Wire Line
-	9000 3600 9000 3450
-Connection ~ 9000 3450
-Wire Wire Line
-	9650 3450 9900 3450
-Wire Wire Line
-	9700 3600 9700 3450
-Connection ~ 9700 3450
-Wire Wire Line
-	10200 3450 10500 3450
-Wire Wire Line
-	6350 5650 6250 5650
-Wire Wire Line
-	2950 1450 2950 1350
-Wire Wire Line
-	2650 1350 4400 1350
-Wire Wire Line
-	3350 1450 3350 1350
-Connection ~ 3350 1350
-Wire Wire Line
-	3750 1450 3750 1350
-Connection ~ 3750 1350
-Wire Wire Line
-	4150 1450 4150 1350
-Connection ~ 4150 1350
-Wire Wire Line
-	3550 3150 3550 4050
-Wire Wire Line
-	3550 3900 3700 3900
-Wire Wire Line
-	4200 3050 4200 4050
-Wire Wire Line
-	4200 3900 4100 3900
-Connection ~ 2650 2350
-Wire Wire Line
-	3550 3150 3300 3150
-Connection ~ 3550 3900
-Wire Wire Line
-	4200 3050 3300 3050
-Connection ~ 4200 3900
-Wire Wire Line
-	4400 2850 3300 2850
-Wire Wire Line
-	3300 2750 4750 2750
-Wire Wire Line
-	4750 2750 4750 2850
-Wire Wire Line
-	3300 3350 5050 3350
-Wire Wire Line
-	3300 3450 5050 3450
-Connection ~ 2950 1350
-Connection ~ 6600 2100
-Wire Wire Line
-	7450 3650 7700 3650
-Wire Wire Line
-	7700 3650 7700 4050
-Wire Wire Line
-	6600 3100 7050 3100
-Connection ~ 6950 3100
-Wire Wire Line
-	6600 3100 6600 2100
-Connection ~ 6850 3100
-Wire Wire Line
-	6350 4250 6350 3750
-Wire Wire Line
-	6350 3750 6450 3750
-Wire Wire Line
-	6100 4250 6100 3650
-Wire Wire Line
-	6100 3650 6450 3650
-Wire Wire Line
-	5850 4250 5850 3550
-Wire Wire Line
-	5850 3550 6450 3550
-Wire Wire Line
-	5400 3350 6450 3350
-Wire Wire Line
-	5400 3450 6450 3450
-Wire Wire Line
-	5100 5650 5150 5650
-Wire Wire Line
-	5100 3750 5100 5650
-Wire Wire Line
-	4900 5850 5150 5850
-Wire Wire Line
-	4900 3000 4900 5850
-Wire Wire Line
-	4900 3000 5350 3000
-Wire Wire Line
-	5950 5850 6700 5850
-Wire Wire Line
-	2650 1350 2650 2350
-Wire Wire Line
-	1900 3350 2000 3350
-Wire Wire Line
-	2000 3250 1900 3250
-Wire Wire Line
-	1900 3150 2000 3150
-Wire Wire Line
-	2000 3550 2000 3550
-Wire Wire Line
-	1900 3450 2000 3450
-Wire Wire Line
-	5750 4850 6350 4850
-Wire Wire Line
-	6350 4850 6350 4550
-Wire Wire Line
-	5750 4750 6100 4750
-Wire Wire Line
-	6100 4750 6100 4550
-Wire Wire Line
-	5750 4650 5850 4650
-Wire Wire Line
-	5850 4650 5850 4550
-Wire Wire Line
-	2550 2350 2750 2350
 $Comp
 L GND #PWR023
@@
 	1    0    0    -1
 $EndComp
-Wire Wire Line
-	1250 2950 2000 2950
-Wire Wire Line
-	1350 2950 1350 3350
-Wire Wire Line
-	5550 1350 5000 1350
-Wire Wire Line
-	5000 2100 5150 2100
 Text HLabel 1250 2950 0    60   Output ~ 0
 SFD
@@
 	1    0    0    -1
 $EndComp
-Wire Wire Line
-	900  3350 900  2650
-Wire Wire Line
-	800  2650 2000 2650
-Connection ~ 1350 2950
 Text HLabel 800  2650 0    60   Output ~ 0
 FIFO
-Connection ~ 900  2650
 Text HLabel 1250 2750 0    60   Output ~ 0
 FIFOP
 Text HLabel 1250 2850 0    60   Output ~ 0
 CCA
-Wire Wire Line
-	1250 2850 2000 2850
-Wire Wire Line
-	2000 2750 1250 2750
 $Comp
 L LED D1
@@
 	1    0    0    -1
 $EndComp
+Text Label 6250 2100 0    60   ~ 0
+VDD_CC2592_ISO
+Text Label 2550 1350 0    60   ~ 0
+VDD_CC2520_ISO
+Wire Wire Line
+	5750 2100 8100 2100
+Wire Wire Line
+	6000 2100 6000 2150
+Wire Wire Line
+	7650 2100 7650 2150
+Connection ~ 6000 2100
+Wire Wire Line
+	7050 2150 7050 2100
+Connection ~ 7050 2100
+Wire Wire Line
+	7350 2150 7350 2100
+Connection ~ 7350 2100
+Wire Wire Line
+	8100 2100 8100 2700
+Connection ~ 7650 2100
+Wire Wire Line
+	8100 3300 8100 3600
+Wire Wire Line
+	7450 3450 8300 3450
+Connection ~ 8100 3450
+Wire Wire Line
+	8900 3450 9050 3450
+Wire Wire Line
+	9000 3600 9000 3450
+Connection ~ 9000 3450
+Wire Wire Line
+	9650 3450 9900 3450
+Wire Wire Line
+	9700 3600 9700 3450
+Connection ~ 9700 3450
+Wire Wire Line
+	10200 3450 10500 3450
+Wire Wire Line
+	6350 5650 6250 5650
+Wire Wire Line
+	2950 1450 2950 1350
+Wire Wire Line
+	2550 1350 4400 1350
+Wire Wire Line
+	3350 1450 3350 1350
+Connection ~ 3350 1350
+Wire Wire Line
+	3750 1450 3750 1350
+Connection ~ 3750 1350
+Wire Wire Line
+	4150 1450 4150 1350
+Connection ~ 4150 1350
+Wire Wire Line
+	3550 3150 3550 4050
+Wire Wire Line
+	3550 3900 3700 3900
+Wire Wire Line
+	4200 3050 4200 4050
+Wire Wire Line
+	4200 3900 4100 3900
+Wire Wire Line
+	3550 3150 3300 3150
+Connection ~ 3550 3900
+Wire Wire Line
+	4200 3050 3300 3050
+Connection ~ 4200 3900
+Wire Wire Line
+	4400 2850 3300 2850
+Wire Wire Line
+	3300 2750 4750 2750
+Wire Wire Line
+	4750 2750 4750 2850
+Wire Wire Line
+	3300 3350 5050 3350
+Wire Wire Line
+	3300 3450 5050 3450
+Connection ~ 2950 1350
+Connection ~ 6600 2100
+Wire Wire Line
+	7450 3650 7700 3650
+Wire Wire Line
+	7700 3650 7700 4050
+Wire Wire Line
+	6600 3100 7050 3100
+Connection ~ 6950 3100
+Wire Wire Line
+	6600 3100 6600 2100
+Connection ~ 6850 3100
+Wire Wire Line
+	6350 4250 6350 3750
+Wire Wire Line
+	6350 3750 6450 3750
+Wire Wire Line
+	6100 4250 6100 3650
+Wire Wire Line
+	6100 3650 6450 3650
+Wire Wire Line
+	5850 4250 5850 3550
+Wire Wire Line
+	5850 3550 6450 3550
+Wire Wire Line
+	5400 3350 6450 3350
+Wire Wire Line
+	5400 3450 6450 3450
+Wire Wire Line
+	5100 5650 5150 5650
+Wire Wire Line
+	5100 3750 5100 5650
+Wire Wire Line
+	4900 5850 5150 5850
+Wire Wire Line
+	4900 3000 4900 5850
+Wire Wire Line
+	5950 5850 6700 5850
+Wire Wire Line
+	1900 3350 2000 3350
+Wire Wire Line
+	2000 3250 1900 3250
+Wire Wire Line
+	1900 3150 2000 3150
+Wire Wire Line
+	2000 3550 2000 3550
+Wire Wire Line
+	1900 3450 2000 3450
+Wire Wire Line
+	5750 4850 6350 4850
+Wire Wire Line
+	6350 4850 6350 4550
+Wire Wire Line
+	5750 4750 6100 4750
+Wire Wire Line
+	6100 4750 6100 4550
+Wire Wire Line
+	5750 4650 5850 4650
+Wire Wire Line
+	5850 4650 5850 4550
+Wire Wire Line
+	1250 2950 2000 2950
+Wire Wire Line
+	1350 2950 1350 3350
+Wire Wire Line
+	5550 1350 5000 1350
+Wire Wire Line
+	5000 2100 5150 2100
+Wire Wire Line
+	900  3350 900  2650
+Wire Wire Line
+	800  2650 2000 2650
+Connection ~ 1350 2950
+Connection ~ 900  2650
+Wire Wire Line
+	1250 2850 2000 2850
+Wire Wire Line
+	2000 2750 1250 2750
 Wire Wire Line
 	2000 3050 1500 3050
@@
 	1500 3050 1500 3100
 Wire Wire Line
-	5100 3750 5350 3750
-Wire Wire Line
-	5350 3000 5350 3050
+	5100 3050 5100 3000
+Wire Wire Line
+	5100 3000 4900 3000
+Wire Wire Line
+	2550 1350 2550 2350
+Wire Wire Line
+	2450 2350 3050 2350
+Connection ~ 2550 2350
+Connection ~ 2650 2350
+Connection ~ 2750 2350
+Connection ~ 2850 2350
+Connection ~ 2950 2350
 $EndSCHEMATC

Commit message: Mostly finished up 900MHz routing.
Connections:
- net at C6.1: now also U1.27 (DCOUPL)
- net at R1.1: now also U1.23 (RBIAS)
Changed lines of the file:
@@
 Connection ~ 2850 2350
 Connection ~ 2950 2350
+Wire Wire Line
+	3300 2850 3300 2900
+Wire Wire Line
+	3300 2800 3300 2750
 $EndSCHEMATC

Commit message: Silk cleanup and some more routing finessing.
Connections:
- net ANT1_50: now reaches C13.1, L3.1, L4.1, U2.10 (ANT)
- net ANT2_50: now reaches C14.1, L4.2, L5.1
- net ANT3_50: now reaches C15.1, C16.2, L5.2
- net ANT4_50: now reaches C16.1, P2.1 (In)
- net RF_P: now reaches R7.2, U1.17 (RF_P)
- net RF_N: now reaches R6.2, U1.19 (RF_N)
- net RF1_N: now reaches R6.1, U2.2 (RF_N)
- net RF1_P: now reaches R7.1, U2.3 (RF_P)
- net RF2_P: now reaches R7.3, U5.4 (BALP)
- net RF2_N: now reaches R6.3, U5.6 (BALN)
- net ANT5_50: now reaches P1.1 (In), U5.1 (UNBAL)
Changed lines of the file:
@@
 Wire Wire Line
 	3300 2800 3300 2750
+Text Label 3700 3350 0    60   ~ 0
+RF_N
+Text Label 3700 3450 0    60   ~ 0
+RF_P
+Text Label 5750 3350 0    60   ~ 0
+RF1_N
+Text Label 5750 3450 0    60   ~ 0
+RF1_P
+Text Label 5100 4200 1    60   ~ 0
+RF2_P
+Text Label 4900 4200 1    60   ~ 0
+RF2_N
+Text Label 7650 3450 0    60   ~ 0
+ANT1_50
+Text Label 9000 3450 1    60   ~ 0
+ANT2_50
+Text Label 9700 3450 1    60   ~ 0
+ANT3_50
+Text Label 10300 3450 1    60   ~ 0
+ANT4_50
+Text Label 6600 5850 1    60   ~ 0
+ANT5_50
 $EndSCHEMATC
