File: 2G4Radio.sch (KiCad schematic (older format))
At the start: 38 parts, among them P1 BNC, P2 BNC, U1 CC2520, U2 CC2592, U5 LDB182G4520C-110, X1 FA-20H32.0000MF20X-K3

Commit message: Added 3.3V LDO
Parts:
- renumbered C7 to C6, C6 to C7, L1 to L2, L2 to L3, L3 to L4, L4 to L5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
